File: Hardware/kicad4ADSb0.1andChildBoard/ADSb0.1andChildBoard/ADSb0.1andChildBoard.sch (KiCad schematic (older format))
At the start: 18 parts, among them IC1 AD7856ANZ, J1 ICSP ARDUINO NANO, J2 Conn_01x04, J3 Conn_01x04, J4 Conn_01x04, J5 Conn_01x04, J6 Conn_01x04, J7 Conn_01x04, U1 MAX7375AXR405

Commit message: Kicad mockup
Kicad mockup
Parts:
- removed C1, C6: 0.01e-6, Capacitor_Tantalum_SMD:CP_EIA-2012-12_Kemet-R_Pad1.30x1.05mm_HandSolder, symbol Device:CP1_Small
- removed C2: 10e-6, Capacitor_Tantalum_SMD:CP_EIA-2012-12_Kemet-R_Pad1.30x1.05mm_HandSolder, symbol Device:CP1_Small
- removed C3, C5, C7, C8: 0.1e-6, Capacitor_Tantalum_SMD:CP_EIA-2012-12_Kemet-R_Pad1.30x1.05mm_HandSolder, symbol Device:CP1_Small
- removed C4: 470e-9, Capacitor_Tantalum_SMD:CP_EIA-2012-12_Kemet-R_Pad1.30x1.05mm_HandSolder, symbol Device:CP1_Small
- removed IC1: AD7856ANZ, Package_SO:SOIC-24W_7.5x15.4mm_P1.27mm, symbol SamacSys_Parts:AD7856ANZ
- removed R1: 10, Resistor_SMD:R_1206_3216Metric, symbol Device:R_Small
- removed U1: MAX7375AXR405, Package_TO_SOT_SMD:SOT-323_SC-70, symbol Oscillator:MAX7375AXR405
- added J8: Conn_02x09_Counter_Clockwise, Connector_Molex:Molex_Picoflex_90325-0018_2x09_P1.27mm_Vertical, symbol Connector_Generic:Conn_02x09_Counter_Clockwise
Connections:
- wire segments 123 -> 111
