File: Hardware/kicad4ADSb0.1/ADSSBb0.1/ADSSBb0.1.kicad_pcb (KiCad board)
At the start: 2 copper layers, 18 parts, among them IC1 AD7856ANZ, J1 ICSP ARDUINO NANO, J2 Conn_01x04, J3 Conn_01x04, J4 Conn_01x04, J5 Conn_01x04, J6 Conn_01x04, J7 Conn_01x04, U1 MAX7375AXR405

Commit message: Kicad mockup
Kicad mockup
Parts:
- C1, C2, C3, C4, C6, C7, C8: footprint Capacitor_THT:CP_Radial_D4.0mm_P1.50mm -> Capacitor_Tantalum_SMD:CP_EIA-2012-12_Kemet-R_Pad1.30x1.05mm_HandSolder
- C5: footprint Capacitor_THT:CP_Radial_D4.0mm_P1.50mm -> Capacitor_Tantalum_SMD:CP_EIA-2012-12_Kemet-R_Pad1.30x1.05mm_HandSolder; moved to F.Cu
- IC1: footprint Package_DIP:DIP-24_W10.16mm -> Package_SO:SOIC-24W_7.5x15.4mm_P1.27mm; moved to F.Cu
- R1: footprint Resistor_THT:R_Axial_DIN0204_L3.6mm_D1.6mm_P1.90mm_Vertical -> Resistor_SMD:R_1206_3216Metric
- moved J2 63.0 mm to (161.3, 67.3)
- moved C7 49.5 mm to (133.3, 67.3)
- moved J3 48.4 mm to (161.3, 85.1)
- moved J1 44.0 mm to (168.9, 78.7)
- moved R1 41.4 mm to (123.2, 67.3)
- moved C8 40.6 mm to (138.4, 67.3)
- moved J6 35.2 mm to (152.4, 72.4), turned to 0 degrees
- moved C4 32.5 mm to (137.2, 85.1)
- moved C1 32.5 mm to (128.3, 67.3)
- moved IC1 30.7 mm to (132.1, 76.2)
- moved C5 29.6 mm to (141.9, 85.1)
- moved J4 28.5 mm to (160.0, 72.4), turned to 0 degrees
- moved J7 27.9 mm to (148.6, 80.0), turned to 180 degrees
- moved U1 27.1 mm to (121.7, 84.5)
- moved C6 26.7 mm to (132.1, 85.1)
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
Commit message: Kicad up
Parts:
- moved J1 65.9 mm to (118.1, 120.7)
- moved J6 57.3 mm to (156.2, 129.5), turned to 270 degrees
- moved J2 53.3 mm to (156.2, 120.4), turned to 270 degrees
- moved J4 52.7 mm to (156.2, 125.0), turned to 270 degrees
- moved IC1 41.9 mm to (130.8, 118.1)
- moved J5 38.9 mm to (156.2, 111.3), turned to 270 degrees
- moved J3 31.2 mm to (156.2, 115.8), turned to 270 degrees
- moved J7 27.7 mm to (156.2, 106.7), turned to 270 degrees
Other:
- board outline added: 43.7 x 17.8 mm

Commit message: Up Kicad
Parts:
- moved C4 43.4 mm to (125.8, 127.0)
- moved C6 43.4 mm to (120.7, 127.0)
- moved C3 43.4 mm to (136.2, 127.0)
- moved C5 43.4 mm to (130.8, 127.0)
- moved C7 42.4 mm to (139.4, 109.2)
- moved C8 42.1 mm to (134.6, 109.2)
- moved C1 41.9 mm to (129.8, 109.2)
- moved R1 41.9 mm to (123.6, 109.2)
- moved U1 26.9 mm to (117.1, 111.0), turned to 90 degrees
- moved C2 20.9 mm to (123.2, 105.7)
Routing:
- net /5V: track 0.00 -> 136.7 mm, vias 0 -> 1
- net GND: track 0.00 -> 128.8 mm
- net Net-(C3-Pad1): track 0.00 -> 46.5 mm
- net Net-(IC1-Pad13): track 0.00 -> 33.5 mm
- net Net-(IC1-Pad9): track 0.00 -> 21.6 mm
- net Net-(IC1-Pad10): track 0.00 -> 19.8 mm
- net Net-(C7-Pad1): track 0.00 -> 19.3 mm
- net Net-(IC1-Pad12): track 0.00 -> 19.0 mm, vias 0 -> 1
- net Net-(IC1-Pad14): track 0.00 -> 18.4 mm
- net Net-(C6-Pad1): track 0.00 -> 18.4 mm
- net /SCK: track 0.00 -> 17.6 mm
- net Net-(IC1-Pad11): track 0.00 -> 16.8 mm
- net /MOSI: track 0.00 -> 16.0 mm
- net /MISO: track 0.00 -> 14.6 mm
- net Net-(C4-Pad1): track 0.00 -> 10.6 mm
- added copper zone on B.Cu, net GND
Other:
- board size 43.7 x 17.8 mm -> 43.7 x 27.4 mm

Commit message: kicad rup
Parts:
- moved J1 5.68 mm to (115.6, 115.6), turned to 180 degrees
Routing:
- net GND: track 128.8 -> 137.8 mm
- net /MOSI: track 16.0 -> 11.9 mm
- net /MISO: track 14.6 -> 18.2 mm, vias 0 -> 1
- net /5V: track 136.7 -> 134.0 mm
- net /SCK: track 17.6 -> 19.7 mm

Commit message: Ricad
New PCB
Parts:
- added J8: Conn_01x03, Connector_PinHeader_2.54mm:PinHeader_1x03_P2.54mm_Vertical, F.Cu at (137.2, 129.5)
Routing:
- net GND: track 137.8 -> 15.0 mm, vias 0 -> 12
- net Net-(C3-Pad1): track 46.5 -> 73.4 mm
- net Net-(IC1-Pad15): track 0.00 -> 21.9 mm, vias 0 -> 1
- net Net-(C7-Pad1): track 19.3 -> 36.0 mm, vias 0 -> 2
- net Net-(IC1-Pad10): track 19.8 -> 33.6 mm, vias 0 -> 1
- net /SCK: track 19.7 -> 27.6 mm
- net /5V: track 134.0 -> 128.6 mm, vias 1 -> 0
- net /MOSI: track 11.9 -> 14.9 mm
- net Net-(IC1-Pad9): track 21.6 -> 24.0 mm
- net Net-(IC1-Pad13): track 33.5 -> 35.5 mm
- net /MISO: track 18.2 -> 16.7 mm
- net Net-(IC1-Pad11): track 16.8 -> 18.1 mm, vias 0 -> 1
- net Net-(IC1-Pad12): track 19.0 -> 18.3 mm, vias 1 -> 0
- net Net-(IC1-Pad14): vias 0 -> 1
Other:
- outline, holes or cut-outs redrawn
- net class POWER added: clearance 0.25, trace_width 0.5, via_dia 0.8, via_drill 0.4
