File: Hardware/kicad4ADSb0.1/ADSSBb0.1/ADSSBb0.1.sch (KiCad schematic (older format))
At the start: 18 parts, among them IC1 AD7856ANZ, J1 ICSP ARDUINO NANO, J2 Conn_01x04, J3 Conn_01x04, J4 Conn_01x04, J5 Conn_01x04, J6 Conn_01x04, J7 Conn_01x04, U1 MAX7375AXR405

Commit message: Ricad
New PCB
Parts:
- added J8: Conn_01x03, Connector_PinHeader_2.54mm:PinHeader_1x03_P2.54mm_Vertical, symbol Connector_Generic:Conn_01x03
Connections:
- net 5V: now also J8.1 (Pin_1)
- net GND: now also J8.3 (Pin_3)
- net at IC1.15 (AIN7): now also J8.2 (Pin_2)
